File: Practiques/Practica 1/Exemple1/Exemple_1/Exemple_1.kicad_pcb (KiCad board)
At the start: 2 copper layers, 58.4 x 20.3 mm, 11 parts, among them J1 Cin, U1 NE555P

Commit message: Posada_a_Punt
Routing:
- net Net-(D1-K): track 0.00 -> 6.16 mm
Changed lines of the file:
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@@
         (effects (font (size 1 1) (thickness 0.15)))
     )
-    (fp_text value "MountingHole_2mm" (at 0 3.1) (layer "F.Fab")
+    (fp_text value "MountingHole_2mm" (at 0 3.1) (layer "F.Fab") hide
         (effects (font (size 1 1) (thickness 0.15)))
     )
@@
         (effects (font (size 1 1) (thickness 0.15)))
     )
-    (fp_text value "6k8" (at 0 -1.4625 90) (layer "F.Fab")
+    (fp_text value "6k8" (at 0 -2.4625 90) (layer "F.Fab")
         (effects (font (size 1 1) (thickness 0.15)))
     )
@@
     (property "ki_keywords" "R res resistor")
     (attr smd)
-    (fp_text reference "R2" (at 0 2.8575 90) (layer "B.Cu")
-        (effects (font (size 1 1) (thickness 0.15)))
-    )
-    (fp_text value "18k" (at 0 -1.4625 90) (layer "F.Fab")
+    (fp_text reference "R2" (at 0 2.8575 90) (layer "F.SilkS")
+        (effects (font (size 1 1) (thickness 0.15)))
+    )
+    (fp_text value "18k" (at 0 -2.4625 90) (layer "F.Fab")
         (effects (font (size 1 1) (thickness 0.15)))
     )
@@
         (effects (font (size 1 1) (thickness 0.15)))
     )
-    (fp_text value "MountingHole_2mm" (at 0 3.1) (layer "F.Fab")
+    (fp_text value "MountingHole_2mm" (at 0 3.1) (layer "F.Fab") hide
         (effects (font (size 1 1) (thickness 0.15)))
     )
@@
         (effects (font (size 1 1) (thickness 0.15)))
     )
-    (fp_text value "220" (at 0 1.82 90) (layer "F.Fab")
+    (fp_text value "220" (at 0 2.82 90) (layer "F.Fab")
         (effects (font (size 1 1) (thickness 0.15)))
     )
@@
         (effects (font (size 1 1) (thickness 0.15)))
     )
-    (fp_text value "MountingHole_2mm" (at 0 3.1) (layer "F.Fab")
+    (fp_text value "MountingHole_2mm" (at 0 3.1) (layer "F.Fab") hide
         (effects (font (size 1 1) (thickness 0.15)))
     )
@@
         (effects (font (size 1 1) (thickness 0.15)))
     )
-    (fp_text value "MountingHole_2mm" (at 0 3.1) (layer "F.Fab")
+    (fp_text value "MountingHole_2mm" (at 0 3.1) (layer "F.Fab") hide
         (effects (font (size 1 1) (thickness 0.15)))
     )
@@
   (segment (start 121.92 83.82) (end 129.56 83.82) (width 0.25) (layer "F.Cu") (net 2))
   (segment (start 109.22 83.82) (end 121.92 83.82) (width 0.25) (layer "F.Cu") (net 2))
+  (segment (start 152.4 83.82) (end 152.4 89.9775) (width 0.25) (layer "F.Cu") (net 3))
+  (segment (start 146.935 81.28) (end 153.672792 81.28) (width 0.5) (layer "F.Cu") (net 4))
+  (segment (start 116.84 88.9) (end 119.38 90.600734) (width 0.5) (layer "F.Cu") (net 4))
+  (segment (start 153.672792 81.28) (end 154.94 82.547208) (width 0.5) (layer "F.Cu") (net 4))
+  (segment (start 119.38 90.600734) (end 130.399266 90.600734) (width 0.5) (layer "F.Cu") (net 4))
+  (segment (start 130.399266 90.600734) (end 130.82 90.18) (width 0.5) (layer "F.Cu") (net 4))
+  (segment (start 138.44 82.56) (end 145.655 82.56) (width 0.5) (layer "F.Cu") (net 4))
   (segment (start 109.22 88.9) (end 116.84 88.9) (width 0.5) (layer "F.Cu") (net 4))
-  (segment (start 146.935 81.28) (end 153.672792 81.28) (width 0.5) (layer "F.Cu") (net 4))
-  (segment (start 118.12 90.18) (end 130.82 90.18) (width 0.5) (layer "F.Cu") (net 4))
-  (segment (start 153.672792 81.28) (end 154.94 82.547208) (width 0.5) (layer "F.Cu") (net 4))
-  (segment (start 116.84 88.9) (end 118.12 90.18) (width 0.5) (layer "F.Cu") (net 4))
-  (segment (start 138.44 82.56) (end 145.655 82.56) (width 0.5) (layer "F.Cu") (net 4))
   (segment (start 145.655 82.56) (end 145.8575 82.3575) (width 0.5) (layer "F.Cu") (net 4))
   (segment (start 145.8575 82.3575) (end 146.935 81.28) (width 0.5) (layer "F.Cu") (net 4))
