File: Practiques/Practica2/AidarIglesias_DavidMiravent_P2-20230312T112003Z-001/AidarIglesias_DavidMiravent_P2/AidarIglesias_DavidMiravent_P2.kicad_pcb (KiCad board)
At the start: 4 copper layers, 30 x 31.3 mm, 17 parts, among them J1 Screw_Terminal_01x02, J2 Conn_01x01_Pin, U1 LT1492, U2 LM1117-ADJ

Commit message: Mod_P3_13_03_23_22_26
Routing:
- net GND: track 40.5 -> 14.6 mm, vias 4 -> 3
- net +VCC: track 32.3 -> 9.63 mm, vias 4 -> 2
Changed lines of the file:
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@@
   (segment (start 113.305 60.205) (end 113.3 60.2) (width 0.5) (layer "F.Cu") (net 4))
   (segment (start 122.8725 54.22) (end 122.8625 54.23) (width 0.5) (layer "F.Cu") (net 4))
-  (segment (start 110.26 64.91) (end 112.17 66.82) (width 0.5) (layer "F.Cu") (net 4))
   (segment (start 131.13 68.37) (end 131.13 65.36) (width 0.5) (layer "F.Cu") (net 4))
   (segment (start 131.1575 62.3225) (end 131.13 62.35) (width 0.5) (layer "F.Cu") (net 4))
   (segment (start 131.13 62.35) (end 131.13 65.36) (width 0.5) (layer "F.Cu") (net 4))
-  (segment (start 118.4 68.085) (end 119.7 66.785) (width 0.5) (layer "F.Cu") (net 4))
-  (segment (start 127 68.58) (end 130.92 68.58) (width 0.5) (layer "F.Cu") (net 4))
-  (segment (start 125.205 66.785) (end 127 68.58) (width 0.5) (layer "F.Cu") (net 4))
-  (segment (start 112.17 66.82) (end 113.435 68.085) (width 0.5) (layer "F.Cu") (net 4))
-  (segment (start 122.1 60.19) (end 123.41 60.19) (width 0.5) (layer "F.Cu") (net 4))
-  (segment (start 109.73 64.25) (end 108.29 62.81) (width 0.5) (layer "F.Cu") (net 4))
   (segment (start 131.1575 60.08) (end 131.1575 62.3225) (width 0.5) (layer "F.Cu") (net 4))
-  (segment (start 113.435 68.085) (end 118.4 68.085) (width 0.5) (layer "F.Cu") (net 4))
   (segment (start 115.215 60.205) (end 113.305 60.205) (width 0.5) (layer "F.Cu") (net 4))
   (segment (start 110.26 64.25) (end 110.26 64.91) (width 0.5) (layer "F.Cu") (net 4))
+  (segment (start 124.57 54.22) (end 122.8725 54.22) (width 0.5) (layer "F.Cu") (net 4))
+  (segment (start 129.76 68.58) (end 130.92 68.58) (width 0.5) (layer "F.Cu") (net 4))
   (segment (start 130.92 68.58) (end 131.13 68.37) (width 0.5) (layer "F.Cu") (net 4))
-  (segment (start 119.7 66.785) (end 125.205 66.785) (width 0.5) (layer "F.Cu") (net 4))
-  (segment (start 123.41 60.19) (end 123.77 59.83) (width 0.5) (layer "F.Cu") (net 4))
-  (segment (start 124.57 54.22) (end 122.8725 54.22) (width 0.5) (layer "F.Cu") (net 4))
   (via (at 124.57 54.22) (size 0.8) (drill 0.4) (layers "F.Cu" "B.Cu") (free) (net 4))
-  (via (at 122.1 60.19) (size 0.8) (drill 0.4) (layers "F.Cu" "B.Cu") (free) (net 4))
-  (via (at 108.29 62.81) (size 0.8) (drill 0.4) (layers "F.Cu" "B.Cu") (free) (net 4))
   (via (at 113.3 60.2) (size 0.8) (drill 0.4) (layers "F.Cu" "B.Cu") (free) (net 4))
+  (via (at 129.76 68.58) (size 0.8) (drill 0.4) (layers "F.Cu" "B.Cu") (free) (net 4))
   (segment (start 115.978249 56.395) (end 119.788249 60.205) (width 0.25) (layer "F.Cu") (net 5))
   (segment (start 115.2275 54.26) (end 115.2275 56.3825) (width 0.25) (layer "F.Cu") (net 5))
@@
   (segment (start 133.855 63.063173) (end 133.855 60.9525) (width 0.25) (layer "F.Cu") (net 6))
   (segment (start 122.205 56.395) (end 122.21 56.4) (width 0.5) (layer "F.Cu") (net 7))
-  (segment (start 129.9 75.58) (end 128.04 75.58) (width 0.5) (layer "F.Cu") (net 7))
-  (segment (start 118.44 75.59) (end 116.24 77.79) (width 0.5) (layer "F.Cu") (net 7))
   (segment (start 110.45873 77.79) (end 108.870001 76.201271) (width 0.5) (layer "F.Cu") (net 7))
   (segment (start 131.02 71.2675) (end 131.1675 71.12) (width 0.5) (layer "F.Cu") (net 7))
   (segment (start 131.16 72.71) (end 131.16 71.1275) (width 0.5) (layer "F.Cu") (net 7))
   (segment (start 133.03 68.37) (end 133.03 69.2575) (width 0.5) (layer "F.Cu") (net 7))
-  (segment (start 128.03 75.59) (end 118.44 75.59) (width 0.5) (layer "F.Cu") (net 7))
   (segment (start 128.04 75.58) (end 128.03 75.59) (width 0.5) (layer "F.Cu") (net 7))
-  (segment (start 116.24 77.79) (end 110.45873 77.79) (width 0.5) (layer "F.Cu") (net 7))
-  (segment (start 108.37 65) (end 108.37 65.52) (width 0.5) (layer "F.Cu") (net 7))
-  (segment (start 108.37 65.52) (end 109.67 66.82) (width 0.5) (layer "F.Cu") (net 7))
   (segment (start 131.16 71.1275) (end 131.1675 71.12) (width 0.5) (layer "F.Cu") (net 7))
   (segment (start 120.165 56.395) (end 122.205 56.395) (width 0.5) (layer "F.Cu") (net 7))
   (segment (start 133.03 69.2575) (end 131.1675 71.12) (width 0.5) (layer "F.Cu") (net 7))
-  (via (at 108.37 65) (size 0.8) (drill 0.4) (layers "F.Cu" "B.Cu") (free) (net 7))
   (via (at 122.21 56.4) (size 0.8) (drill 0.4) (layers "F.Cu" "B.Cu") (free) (net 7))
-  (via (at 129.9 75.58) (size 0.8) (drill 0.4) (layers "F.Cu" "B.Cu") (free) (net 7))
   (via (at 131.16 72.71) (size 0.8) (drill 0.4) (layers "F.Cu" "B.Cu") (free) (net 7))
   (segment (start 113.11 63.27) (end 113.11 64.85) (width 0.5) (layer "F.Cu") (net 8))
