File: Practiques/Practica3/AidarIglesias_DavidMiravent_P3-20230312T223449Z-001/AidarIglesias_DavidMiravent_P3/AidarIglesias_DavidMiravent_P3.kicad_sch (KiCad schematic)
At the start: 32 parts, among them IC1 PIC18F258-I_SO, J1 ANALOG INPUT, J1 Screw_Terminal_01x02, J3 PROGRAMMING CON, J4 JP2, J5 JP1, J6 USART CON, SW1 SW_Push, U1 LM1117-ADJ, U1 LT1492, Y1 ABLS2-16.000MHZ-D4Y-T

Commit message: Mod_13_03_23_22_56
Connections:
- net Vsw: now reaches J5.1 (Pin_1), R6.2, SW1.1
- net Vlb: now reaches D5.1 (K), R8.1
- net Vfbk: now reaches R1.2, R2.1, U1.2 (-)
- net Vled: now reaches D3.1 (K), R5.1
- net Vlr: now reaches D4.1 (K), R7.1
- net Vdd: now reaches D4.2 (A), IC1.20 (VDD)
Changed lines of the file:
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@@
     (stroke (width 0) (type default))
   )
-  (image (at 185.674 43.688)
+  (image (at 214.63 98.552) (scale 1.86799)
     (data
       iVBORw0KGgoAAAANSUhEUgAAAz0AAAKVCAIAAABqMhIVAAAAA3NCSVQICAjb4U/gAAAgAElEQVR4
@@
     (effects (font (size 3 3) bold) (justify left bottom))
   )
+  (label "Vlb" (at 127.762 153.67 0) (fields_autoplaced)
+    (effects (font (size 1.27 1.27)) (justify left bottom))
+  )
+  (label "Vled" (at 132.08 70.866 90) (fields_autoplaced)
+    (effects (font (size 1.27 1.27)) (justify left bottom))
+  )
   (label "V_{in}" (at 60.96 21.59 0) (fields_autoplaced)
+    (effects (font (size 1.27 1.27)) (justify left bottom))
+  )
+  (label "Vfbk" (at 54.102 58.42 0) (fields_autoplaced)
     (effects (font (size 1.27 1.27)) (justify left bottom))
   )
@@
     (effects (font (size 1.27 1.27)) (justify left bottom))
   )
+  (label "Vsw" (at 55.372 121.92 0) (fields_autoplaced)
+    (effects (font (size 1.27 1.27)) (justify left bottom))
+  )
+  (label "Vlr" (at 110.236 168.91 0) (fields_autoplaced)
+    (effects (font (size 1.27 1.27)) (justify left bottom))
+  )
   (label "V_{div}" (at 87.63 30.48 0) (fields_autoplaced)
     (effects (font (size 1.27 1.27)) (justify left bottom))
   )
+  (label "Vdd" (at 100.584 168.91 0) (fields_autoplaced)
+    (effects (font (size 1.27 1.27)) (justify left bottom))
+  )

Commit message: Mod_14_03_23_00_44
Parts:
- D4: footprint LED_SMD:LED_7012X1 -> LED_SMD:LED_0805_2012Metric
- D5: footprint LED_SMD:LEDC2012X70N -> LED_SMD:LED_0805_2012Metric
Connections:
- net Vlb renamed Vledb
- net Vlr renamed Vledr
Changed lines of the file:
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@@
     (stroke (width 0) (type default))
   )
+  (wire (pts (xy 127.254 153.67) (xy 129.032 153.67))
+    (stroke (width 0) (type default))
+  )
   (wire (pts (xy 120.65 111.76) (xy 137.16 111.76))
     (stroke (width 0) (type default))
@@
     (stroke (width 0) (type default))
   )
+  (wire (pts (xy 109.728 168.91) (xy 112.268 168.91))
+    (stroke (width 0) (type default))
+  )
   (wire (pts (xy 59.69 111.76) (xy 59.69 109.22))
     (stroke (width 0) (type default))
@@
     (stroke (width 0) (type default))
   )
-  (wire (pts (xy 127.254 153.67) (xy 129.032 153.67))
-    (stroke (width 0) (type default))
-  )
   (wire (pts (xy 66.04 58.42) (xy 71.12 58.42))
     (stroke (width 0) (type default))
@@
     (stroke (width 0) (type default))
   )
-  (wire (pts (xy 109.728 168.91) (xy 112.268 168.91))
-    (stroke (width 0) (type default))
-  )
   (wire (pts (xy 25.4 36.83) (xy 22.86 36.83))
     (stroke (width 0) (type default))
@@
     (effects (font (size 3 3) bold) (justify left bottom))
   )
-  (label "Vlb" (at 127.762 153.67 0) (fields_autoplaced)
+  (label "Vled" (at 132.08 70.866 90) (fields_autoplaced)
     (effects (font (size 1.27 1.27)) (justify left bottom))
   )
-  (label "Vled" (at 132.08 70.866 90) (fields_autoplaced)
+  (label "Vledr" (at 110.236 168.91 0) (fields_autoplaced)
     (effects (font (size 1.27 1.27)) (justify left bottom))
   )
@@
     (effects (font (size 1.27 1.27)) (justify left bottom))
   )
-  (label "VAMP" (at 73.66 69.85 0) (fields_autoplaced)
+  (label "Vledb" (at 127.762 153.67 0) (fields_autoplaced)
     (effects (font (size 1.27 1.27)) (justify left bottom))
   )
-  (label "Vsw" (at 55.372 121.92 0) (fields_autoplaced)
+  (label "VAMP" (at 73.66 69.85 0) (fields_autoplaced)
     (effects (font (size 1.27 1.27)) (justify left bottom))
   )
-  (label "Vlr" (at 110.236 168.91 0) (fields_autoplaced)
+  (label "Vsw" (at 55.372 121.92 0) (fields_autoplaced)
     (effects (font (size 1.27 1.27)) (justify left bottom))
   )
@@
       (effects (font (size 1.27 1.27)))
     )
-    (property "Footprint" "LED_SMD:LEDC2012X70N" (at 123.444 153.67 0)
+    (property "Footprint" "LED_SMD:LED_0805_2012Metric" (at 123.444 153.67 0)
       (effects (font (size 1.27 1.27)) hide)
     )
@@
       (effects (font (size 1.27 1.27)))
     )
-    (property "Footprint" "LED_SMD:LED_7012X1" (at 105.918 168.91 0)
+    (property "Footprint" "LED_SMD:LED_0805_2012Metric" (at 105.918 168.91 0)
       (effects (font (size 1.27 1.27)) hide)
     )
