File: Practiques/Practica3/DavidMiravent_AidarIglesias_P3/AidarIglesias_DavidMiravent_P3.kicad_pcb (KiCad board)
At the start: 4 copper layers, 56.9 x 45.4 mm, 36 parts, among them IC1 PIC18F258-I_SO, J1 ANALOG INPUT, J2 Screw_Terminal_01x02, J3 PROGRAMMING CON, J4 JP2, J5 JP1, J6 USART CON, SW1 SW_Push, U1 LT1492, U2 LM1117-ADJ, Y1 ABLS2-16.000MHZ-D4Y-T

Commit message: Mod_15_03_23_13_08
Parts:
- moved D5 11.2 mm to (115.9, 112.0)
- moved R8 10.6 mm to (119.7, 112.0)
- moved Y1 1.76 mm to (116.4, 102.5)
- moved C2 1.72 mm to (120.5, 96.5)
- moved C1 1.71 mm to (120.6, 108.7)
Routing:
- net MCLR: track 54.5 -> 64.3 mm
- net PGM: track 6.65 -> 15.3 mm
- net XTAL1: track 21.6 -> 14.4 mm
- net GND: track 26.6 -> 28.0 mm, vias 53 -> 8
- net /VAMP: track 24.0 -> 24.9 mm
- net PGD: track 10.7 -> 11.5 mm
- net /Vledb: track 2.60 -> 1.94 mm
- removed copper zone on F.Cu, net GND
